File: adc.kicad_sch (KiCad schematic)
At the start: 33 parts, among them U1 ADA4945-1, U2 LTC2387-18, U25 ADA4898-2

Commit message: Major schematic and PCB changes and latex manual creation.
Parts:
- added U30: LTC6655BHMS8-4.096#PBF, Package_SO:TSSOP-8_3x3mm_P0.65mm, symbol lib:LTC6655BHMS8-4.096#PBF
- C5, C6: value 82pF -> 180pF; M KEMET -> MURATA; MPN C0402C820J3GACAUTO -> GRT1555C1H181FA02D
Connections:
- net 5VA: now also C9.1, U30.1 (~{SHDN}), U30.2 (V_{IN})
- net GND: now also U2.9 (REFIN), U30.3 (GND), U30.4 (GND), U30.5 (GND), U30.8 (GND)
- net refbuf: now also U30.6 (V_{OUT_S}), U30.7 (V_{OUT_F})
- removed net refin: C9.1, U2.9 (REFIN)
Other:
- note added: "10 MSPS RC filter"
- note added: "500 kHz Bandwidth"
- moved on the sheet: C9
