File: b2b_jb3.kicad_sch (KiCad schematic)
At the start: 11 parts

Commit message: Major schematic and PCB changes and latex manual creation.
Connections:
- net B34_P17: now reaches JB3.19 (P17|B34|T3|L20P)
- net B34_P18: now reaches JB3.21 (P18|B34|T3|L20N)
- net 3V3D_OUT renamed 2V5D
- net B34_L10+ renamed B34_L21
- net B34_L10- renamed B34_L22
- net B34_L15+ renamed B34_M21
- net B34_L15- renamed B34_M22
- net B34_L21+ renamed B34_T16
- net B34_L21- renamed B34_T17
- no-connect marks 15 -> 13
Changed lines of the file:
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@@
 	(title_block
 		(title "4 channel ADC Module")
-		(date "2025-06-03")
+		(date "2025-06-14")
 		(rev "0.1")
 		(company "NOIRLab")
@@
 	(text "MRCC: Multi-Region Clock Capable"
 		(exclude_from_sim no)
-		(at 240.03 95.504 0)
+		(at 239.014 95.504 0)
 		(effects
 			(font
@@
 	)
 	(junction
-		(at 101.6 86.36)
+		(at 101.6 99.06)
 		(diameter 0)
 		(color 0 0 0 0)
 	)
 	(junction
-		(at 101.6 99.06)
+		(at 101.6 101.6)
 		(diameter 0)
 		(color 0 0 0 0)
 	)
 	(junction
-		(at 101.6 101.6)
+		(at 101.6 86.36)
 		(diameter 0)
 		(color 0 0 0 0)
@@
 	)
 	(no_connect
-		(at 208.28 81.28)
-	)
-	(no_connect
 		(at 134.62 119.38)
 	)
@@
 	)
 	(no_connect
-		(at 208.28 78.74)
-	)
-	(no_connect
 		(at 134.62 124.46)
 	)
@@
 	(wire
 		(pts
+			(xy 101.6 83.82) (xy 101.6 86.36)
+		)
+		(stroke
+			(width 0)
+			(type default)
+		)
+	)
+	(wire
+		(pts
 			(xy 83.82 96.52) (xy 90.17 96.52)
 		)
@@
 		)
 	)
+	(global_label "B34_L13-"
+		(shape input)
+		(at 208.28 96.52 0)
+		(fields_autoplaced yes)
+		(effects
+			(font
+				(size 1.27 1.27)
+			)
+			(justify left)
+		)
+		(property "Intersheetrefs" "${INTERSHEET_REFS}"
+			(at 220.9413 96.52 0)
+			(effects
+				(font
+					(size 1.27 1.27)
+				)
+				(justify left)
+				(hide yes)
+			)
+		)
+	)
 	(global_label "3V3D_SYNC"
 		(shape output)
@@
 		)
 	)
-	(global_label "B34_L15-"
-		(shape bidirectional)
+	(global_label "B34_M22"
+		(shape output)
 		(at 208.28 109.22 0)
 		(fields_autoplaced yes)
@@
 		)
 		(property "Intersheetrefs" "${INTERSHEET_REFS}"
-			(at 222.0526 109.22 0)
+			(at 219.7922 109.22 0)
 			(effects
 				(font
@@
 		)
 	)
-	(global_label "B34_L10-"
-		(shape bidirectional)
+	(global_label "B34_L22"
+		(shape output)
 		(at 208.28 88.9 0)
 		(fields_autoplaced yes)
@@
 		)
 		(property "Intersheetrefs" "${INTERSHEET_REFS}"
-			(at 222.0526 88.9 0)
+			(at 219.3689 88.9 0)
 			(effects
 				(font
@@
 		)
 	)
-	(global_label "-15VA_EN"
-		(shape output)
-		(at 134.62 88.9 180)
+	(global_label "B34_L13+"
+		(shape input)
+		(at 208.28 93.98 0)
 		(fields_autoplaced yes)
 		(effects
@@
 				(size 1.27 1.27)
 			)
-			(justify right)
+			(justify left)
 		)
 		(property "Intersheetrefs" "${INTERSHEET_REFS}"
-			(at 123.3496 88.9 0)
+			(at 220.9413 93.98 0)
 			(effects
 				(font
 					(size 1.27 1.27)
 				)
-				(justify right)
+				(justify left)
 				(hide yes)
 			)
 		)
 	)
-	(global_label "B34_L21+"
-		(shape bidirectional)
-		(at 208.28 101.6 0)
+	(global_label "B34_P17"
+		(shape output)
+		(at 208.28 78.74 0)
 		(fields_autoplaced yes)
 		(effects
@@
 		)
 		(property "Intersheetrefs" "${INTERSHEET_REFS}"
-			(at 222.0526 101.6 0)
+			(at 219.6108 78.74 0)
 			(effects
 				(font
@@
 		)
 	)
-	(global_label "4V2A_EN"
+	(global_label "-15VA_EN"
 		(shape output)
-		(at 134.62 104.14 180)
+		(at 134.62 88.9 180)
 		(fields_autoplaced yes)
 		(effects
@@
 		)
 		(property "Intersheetrefs" "${INTERSHEET_REFS}"
-			(at 123.5915 104.14 0)
+			(at 123.3496 88.9 0)
 			(effects
 				(font
@@
 		)
 	)
-	(global_label "B34_L13-"
-		(shape bidirectional)
-		(at 208.28 96.52 0)
+	(global_label "B34_T17"
+		(shape input)
+		(at 208.28 104.14 0)
 		(fields_autoplaced yes)
 		(effects
@@
 		)
 		(property "Intersheetrefs" "${INTERSHEET_REFS}"
-			(at 222.0526 96.52 0)
+			(at 219.3084 104.14 0)
 			(effects
 				(font
@@
 		)
 	)
+	(global_label "4V2A_EN"
+		(shape output)
+		(at 134.62 104.14 180)
+		(fields_autoplaced yes)
+		(effects
+			(font
+				(size 1.27 1.27)
+			)
+			(justify right)
+		)
+		(property "Intersheetrefs" "${INTERSHEET_REFS}"
+			(at 123.5915 104.14 0)
+			(effects
+				(font
+					(size 1.27 1.27)
+				)
+				(justify right)
+				(hide yes)
+			)
+		)
+	)
 	(global_label "5V5A_EN"
 		(shape output)
@@
 		)
 	)
-	(global_label "B34_L10+"
-		(shape bidirectional)
+	(global_label "B34_L21"
+		(shape output)
 		(at 208.28 86.36 0)
 		(fields_autoplaced yes)
@@
 		)
 		(property "Intersheetrefs" "${INTERSHEET_REFS}"
-			(at 222.0526 86.36 0)
+			(at 219.3689 86.36 0)
 			(effects
 				(font
@@
 		)
 	)
-	(global_label "B34_L13+"
-		(shape bidirectional)
-		(at 208.28 93.98 0)
-		(fields_autoplaced yes)
-		(effects
-			(font
-				(size 1.27 1.27)
-			)
-			(justify left)
-		)
-		(property "Intersheetrefs" "${INTERSHEET_REFS}"
-			(at 222.0526 93.98 0)
-			(effects
-				(font
-					(size 1.27 1.27)
-				)
-				(justify left)
-				(hide yes)
-			)
-		)
-	)
 	(global_label "4V2A_PG"
 		(shape input)
@@
 		)
 	)
+	(global_label "B34_P18"
+		(shape output)
+		(at 208.28 81.28 0)
+		(fields_autoplaced yes)
+		(effects
+			(font
+				(size 1.27 1.27)
+			)
+			(justify left)
+		)
+		(property "Intersheetrefs" "${INTERSHEET_REFS}"
+			(at 219.6108 81.28 0)
+			(effects
+				(font
+					(size 1.27 1.27)
+				)
+				(justify left)
+				(hide yes)
+			)
+		)
+	)
 	(global_label "-15V5A_EN"
 		(shape output)
@@
 		)
 	)
-	(global_label "B34_L21-"
-		(shape bidirectional)
-		(at 208.28 104.14 0)
+	(global_label "B34_T16"
+		(shape input)
+		(at 208.28 101.6 0)
 		(fields_autoplaced yes)
 		(effects
@@
 		)
 		(property "Intersheetrefs" "${INTERSHEET_REFS}"
-			(at 222.0526 104.14 0)
+			(at 219.3084 101.6 0)
 			(effects
 				(font
@@
 		)
 	)
-	(global_label "B34_L15+"
-		(shape bidirectional)
+	(global_label "B34_M21"
+		(shape input)
 		(at 208.28 106.68 0)
 		(fields_autoplaced yes)
@@
 		)
 		(property "Intersheetrefs" "${INTERSHEET_REFS}"
-			(at 222.0526 106.68 0)
+			(at 219.7922 106.68 0)
 			(effects
 				(font
@@
 	)
 	(symbol
+		(lib_id "power:+12V")
+		(at 101.6 83.82 0)
+		(unit 1)
+		(exclude_from_sim no)
+		(in_bom yes)
+		(on_board yes)
+		(dnp no)
+		(property "Reference" "#PWR0290"
+			(at 101.6 87.63 0)
+			(effects
+				(font
+					(size 1.27 1.27)
+				)
+				(hide yes)
+			)
+		)
+		(property "Value" "2V5D"
+			(at 101.6 79.756 0)
+			(effects
+				(font
+					(size 1.27 1.27)
+				)
+			)
+		)
+		(property "Footprint" ""
+			(at 101.6 83.82 0)
+			(effects
+				(font
+					(size 1.27 1.27)
+				)
+				(hide yes)
+			)
+		)
+		(property "Datasheet" ""
+			(at 101.6 83.82 0)
+			(effects
+				(font
+					(size 1.27 1.27)
+				)
+				(hide yes)
+			)
+		)
+		(property "Description" "Power symbol creates a global label with name \"+12V\""
+			(at 101.6 83.82 0)
+			(effects
+				(font
+					(size 1.27 1.27)
+				)
+				(hide yes)
+			)
+		)
+		(pin "1"
+		)
+		(instances
+			(project "adc_board_prot"
+				(path "/c6949a33-abae-4c95-a3fe-c6f7de9ef0a5/ee326142-a1ab-40dd-8d19-bfec08848fdc/45f0a0f8-850f-42cf-978a-117b962875a8"
+					(reference "#PWR0290")
+					(unit 1)
+				)
+			)
+		)
+	)
+	(symbol
 		(lib_id "power:GND")
 		(at 208.28 132.08 90)
@@
 					(unit 1)
 				)
-			)
-		)
-	)
-	(symbol
-		(lib_id "power:+3V3")
-		(at 101.6 86.36 0)
-		(unit 1)
-		(exclude_from_sim no)
-		(in_bom yes)
-		(on_board yes)
-		(dnp no)
-		(fields_autoplaced yes)
-		(property "Reference" "#PWR0167"
-			(at 101.6 90.17 0)
-			(effects
-				(font
-					(size 1.27 1.27)
-				)
-				(hide yes)
-			)
-		)
-		(property "Value" "3V3D_OUT"
-			(at 101.6 81.28 0)
-			(effects
-				(font
-					(size 1.27 1.27)
-				)
-			)
-		)
-		(property "Footprint" ""
-			(at 101.6 86.36 0)
-			(effects
-				(font
-					(size 1.27 1.27)
-				)
-				(hide yes)
-			)
-		)
-		(property "Datasheet" ""
-			(at 101.6 86.36 0)
-			(effects
-				(font
-					(size 1.27 1.27)
-				)
-				(hide yes)
-			)
-		)
-		(property "Description" "Power symbol creates a global label with name \"+3V3\""
-			(at 101.6 86.36 0)
-			(effects
-				(font
-					(size 1.27 1.27)
-				)
-				(hide yes)
-			)
-		)
-		(pin "1"
-		)
-		(instances
-			(project "adc_board_prot"
-				(path "/c6949a33-abae-4c95-a3fe-c6f7de9ef0a5/ee326142-a1ab-40dd-8d19-bfec08848fdc/45f0a0f8-850f-42cf-978a-117b962875a8"
-					(reference "#PWR0167")
-					(unit 1)
-				)
