File: clock_gen.kicad_sch (KiCad schematic)
At the start: 22 parts, among them U24 Si5342A-D, Y1 CX3225SB48000D0FLJCC

Commit message: Major schematic and PCB changes and latex manual creation.
Parts:
- removed C147: 6pF, Capacitor_SMD:C_0402_1005Metric, symbol Device:C_Small
- removed C53: 0.1uF, Capacitor_SMD:C_0402_1005Metric, symbol Device:C_Small
- removed R115: 267, Resistor_SMD:R_0402_1005Metric, symbol Device:R_Small
- removed R116: 845, Resistor_SMD:R_0402_1005Metric, symbol Device:R_Small
- added C182, C183: 0.1uF, Capacitor_SMD:C_0402_1005Metric, symbol Device:C_Small
Connections:
- net CLK_SYNC: now also C14.1
- net GND: now also C182.1, C183.1
- net at U24.1 (IN1): now also U24.2 (IN1b), C182.2
- net at U24.10 (IN2): now also U24.11 (IN2b), C183.2
- no-connect marks 16 -> 12
Other:
- note added: "48 MHz Crystal"
- note added: "Floating clock inputs are noise sensitive. Add a cap to non-CMOS unused clock inputs."
- moved on the sheet: C71, C89, R117
