File: misc.kicad_sch (KiCad schematic)
At the start: 5 parts, among them U23 24LC16BT-I/OT

Commit message: edit README.md
Other:
- company: (none) -> NOIRLab
- title: (none) -> 4 channel ADC Module
Changed lines of the file:
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@@
 	(generator_version "9.0")
 	(paper "A4")
+	(title_block
+		(title "4 channel ADC Module")
+		(date "2025-04-18")
+		(rev "0.1")
+		(company "NOIRLab")
+		(comment 1 "Design: Braulio Cancino Vera - braulio.cancino@noirlab.edu")
+	)
 	(rectangle
 		(start 24.13 22.86)
