File: power_2v5a.kicad_sch (KiCad schematic)
At the start: 10 parts, among them U14 LT3045

Commit message: edit README.md
Other:
- company: (none) -> NOIRLab
- title: (none) -> 4 channel ADC Module
Changed lines of the file:
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@@
 	(generator_version "9.0")
 	(paper "A4")
+	(title_block
+		(title "4 channel ADC Module")
+		(date "2025-04-18")
+		(rev "0.1")
+		(company "NOIRLab")
+		(comment 1 "Design: Braulio Cancino Vera - braulio.cancino@noirlab.edu")
+	)
 	(text "OUTS and SET GND kelvin \nconnected to output capacitor\nto improve PSRR"
 		(exclude_from_sim no)
